File: Hardware/kicad-files-usb/dabao_v3c.kicad_pcb (KiCad board)
At the start: 2 copper layers, 21 x 48.5 mm, 45 parts, among them J1 USB_A, SW1 SW_Push, U1 EMS4000RSW, U2 baochip1x, U3 MT3406, U4 MT3406, Y1 48.000MHz

Commit message: updated files
Routing:
- net /EN: track 47.0 -> 41.8 mm
- net +0.9V: track 30.7 -> 28.2 mm
- net /RST_N: track 37.0 -> 34.5 mm
- net GND: vias 74 -> 79

Commit message: updated files
Other:
- board text added: "3.3V"
Changed lines of the file:
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@@
+		)
+	)
+	(gr_text "3.3V"
+		(at 136.4 79.6 0)
+		(layer "B.SilkS")
+		(effects
+			(font
+				(size 1 1)
+				(thickness 0.1)
+			)
+			(justify left bottom mirror)
 		)
 	)
