File: Hardware/kicad-sd-card/dabao_v3c_sdcard.kicad_pcb (KiCad board)
At the start: 2 copper layers, 21 x 67.5 mm, 44 parts, among them J1 USB_A, J2 Micro_SD_Card, SW1 SW_Push, U1 EMS4000RSW, U2 baochip1x, U3 MT3406, U4 MT3406, U5 CM1624, Y1 48.000MHz

Commit message: Update SD card KiCad PCB layout for dabao_v3c_sdcard.
Syncs local board edits that were not included in the prior hardware push.

Co-authored-by: Cursor <cursoragent@cursor.com>
Routing:
- net +0.9V: track 32.1 -> 31.1 mm
- net GND: track 67.8 -> 66.9 mm, vias 89 -> 114
Other:
- board text added: "3.3V"
